File: RndSeq.kicad_pcb (KiCad board)
At the start: 2 copper layers, 39.6 x 100 mm, 92 parts, among them J1 Conn_01x03, J2 Conn_02x03_Odd_Even, J3 Conn_01x03, J4 Conn_02x05_Odd_Even, SW1 SW_SPDT_MSM, SW2 SW_SPDT_MSM, SW3 SW_SPDT_MSM, SW4 SW_SPDT_MSM, SW5 SW_SPDT_MSM, SW6 SW_Push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

Commit message: Placement in progress...
Parts:
- SW6: moved to F.Cu
- U3: footprint Package_TO_SOT_THT:TO-220-3_Horizontal_TabDown -> Local:TO-220-3_NoHole
- moved C18 150.9 mm to (105.6, 75.8)
- moved C20 150.9 mm to (117.5, 75.1)
- moved C21 150.9 mm to (117.5, 73.1)
- moved C22 150.9 mm to (112.4, 75.8)
- moved C19 150.9 mm to (116.2, 80.7)
- moved R10 143.9 mm to (105.2, 42.9)
- moved R13 142.1 mm to (105.6, 58.8)
- moved R12 138.8 mm to (105.2, 53.7)
- moved R1 137.2 mm to (93.8, 95.6)
- moved R14 134.9 mm to (104.6, 64.5)
- moved R5 133.2 mm to (93.2, 117.2)
- moved C1 132.0 mm to (95.4, 87.4)
- moved R3 131.4 mm to (93.2, 107.0)
- moved C2 127.2 mm to (105.9, 35.3)
- moved R11 124.2 mm to (105.9, 48.6)
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Connections:
- C1 pad 2: GND -> (no net)
- C10 pad 2: GND -> (no net)
- C13 pad 1: GND -> (no net)
- C14 pad 2: GND -> (no net)
- C15 pad 1: GND -> (no net)
- C16 pad 1: GND -> (no net)
- C17 pad 1: GND -> (no net)
- C18 pad 2: GND -> (no net)
- C19 pad 1: GND -> (no net)
- C2 pad 2: GND -> (no net)
- C20 pad 2: GND -> (no net)
- C21 pad 2: GND -> (no net)
- C22 pad 2: GND -> (no net)
- C3 pad 2: GND -> (no net)
- C4 pad 2: GND -> (no net)
- C5 pad 2: GND -> (no net)
- C6 pad 2: GND -> (no net)
- C7 pad 2: GND -> (no net)
- C8 pad 1: GND -> (no net)
- C9 pad 2: GND -> (no net)
- D12 pad 1: GND -> (no net)
- D2 pad 2: GND -> (no net)
- D4 pad 2: GND -> (no net)
- D5 pad 1: GND -> (no net)
- D6 pad 1: GND -> (no net)
- D7 pad 1: GND -> (no net)
- D8 pad 1: GND -> (no net)
- D9 pad 1: GND -> (no net)
- J-CV1 pad S: GND -> (no net)
- J-CV1 pad TN: GND -> (no net)
- J-Clk1 pad S: GND -> (no net)
- J-Out1 pad S: GND -> (no net)
- J-Trig1 pad S: GND -> (no net)
- J1 pad 1: GND -> (no net)
- J2 pad 6: GND -> (no net)
- J3 pad 1: GND -> (no net)
- J4 pad 3: GND -> (no net)
- J4 pad 4: GND -> (no net)
- J4 pad 5: GND -> (no net)
- J4 pad 6: GND -> (no net)
- J4 pad 7: GND -> (no net)
- J4 pad 8: GND -> (no net)
- R30 pad 1: GND -> (no net)
- R31 pad 1: GND -> (no net)
- R34 pad 2: GND -> (no net)
- R35 pad 2: GND -> (no net)
- RV1 pad 3: GND -> (no net)
- SW1 pad 2: GND -> (no net)
- SW2 pad 2: GND -> (no net)
- SW3 pad 2: GND -> (no net)
- SW4 pad 2: GND -> (no net)
- SW5 pad 2: GND -> (no net)
- SW6 pad 2: GND -> (no net)
- U2 pad 21: GND -> (no net)
- U2 pad 5: GND -> (no net)
- U3 pad 2: GND -> (no net)

Commit message: Routed all signals.
Parts:
- moved SW6 103.5 mm to (143.8, 148.2)
- moved C1 68.6 mm to (161.1, 67.7), turned to 90 degrees
- moved R1 65.9 mm to (153.5, 67.7), turned to 270 degrees
- moved R3 63.5 mm to (152.8, 85.4), turned to 270 degrees
- moved R14 62.7 mm to (152.8, 104.5), turned to 90 degrees
- moved C2 61.9 mm to (161.1, 63.2), turned to 270 degrees
- moved R5 60.3 mm to (152.8, 108.9), turned to 270 degrees
- moved R38 60.2 mm to (137.0, 93.7), turned to 90 degrees
- moved R13 58.1 mm to (141.4, 104.5), turned to 270 degrees
- moved C13 57.5 mm to (141.0, 100.4), turned to 90 degrees
- moved C18 56.7 mm to (162.4, 76.6)
- moved C15 56.2 mm to (144.8, 104.5), turned to 90 degrees
- moved R12 55.0 mm to (152.8, 81.3), turned to 90 degrees
- moved R10 52.4 mm to (153.5, 63.2), turned to 90 degrees
- moved R2 49.6 mm to (141.4, 87.4), turned to 90 degrees
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Routing:
- net Net-(C11-Pad1): track 0.00 -> 124.3 mm
- net /MCU328/PD4: track 0.00 -> 90.5 mm
- net Net-(J2-Pad5): track 0.00 -> 88.1 mm, vias 0 -> 5
- net /MCU328/PC3: track 0.00 -> 86.8 mm
- net /MCU328/PD7: track 0.00 -> 79.1 mm
- net /MCU328/PD6: track 0.00 -> 55.2 mm
- net /MCU328/PC2: track 0.00 -> 54.8 mm, vias 0 -> 2
- net /MCU328/PC0: track 0.00 -> 51.4 mm, vias 0 -> 2
- net /MCU328/PB0: track 0.00 -> 51.1 mm
- net Net-(R3-Pad2): track 0.00 -> 49.5 mm, vias 0 -> 4
- net /MCU328/PD5: track 0.00 -> 46.5 mm
- net /MCU328/PD3: track 0.00 -> 41.8 mm, vias 0 -> 4
- net +5V: track 0.00 -> 41.6 mm
- net /MCU328/PC1: track 0.00 -> 39.8 mm
- net Net-(R12-Pad2): track 0.00 -> 36.3 mm, vias 0 -> 2
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Other:
- net class Default: clearance 0.2 -> 0.254; trace_width 0.25 -> 0.254
- rule trace_clearance: 0.2 -> 0.254

Commit message: Routed all power.
Routing:
- net +5V: track 41.6 -> 274.5 mm, vias 0 -> 4
- net -12V: track 9.70 -> 88.5 mm, vias 0 -> 2
- net +12V: track 36.2 -> 94.9 mm, vias 0 -> 2
- net Net-(J2-Pad3): track 32.6 -> 28.0 mm
- net Net-(C10-Pad1): track 15.5 -> 17.7 mm
- net Net-(C11-Pad1): track 124.3 -> 122.3 mm
- net Net-(J2-Pad5): track 88.1 -> 89.5 mm
- net /MCU328/PD4: track 90.5 -> 91.7 mm
- net /MCU328/PC3: track 86.8 -> 87.8 mm
- net Net-(C12-Pad1): track 33.1 -> 32.4 mm
- net /MCU328/PD3: track 41.8 -> 41.2 mm
- net Net-(R3-Pad2): track 49.5 -> 50.0 mm

Commit message: Tidy up tracks.
Routing:
- net +5V: track 274.5 -> 280.0 mm
- net -12V: track 88.5 -> 93.3 mm
- net Net-(C11-Pad1): track 122.3 -> 119.0 mm
- net +12V: track 94.9 -> 97.6 mm
- net /MCU328/PD4: track 91.7 -> 92.4 mm
- net /MCU328/PB0: track 51.1 -> 50.5 mm
- net Net-(J2-Pad4): track 30.1 -> 29.6 mm

Commit message: Finished routing.
Parts:
- U3: footprint Local:TO-220-3_NoHole -> Package_TO_SOT_THT:TO-220-3_Vertical
- renumbered J1 to I2C, J2 to ISP, J3 to SERIAL
Connections:
- C1 pad 2: (no net) -> GND
- C10 pad 2: (no net) -> GND
- C13 pad 1: (no net) -> GND
- C14 pad 2: (no net) -> GND
- C15 pad 1: (no net) -> GND
- C16 pad 1: (no net) -> GND
- C17 pad 1: (no net) -> GND
- C18 pad 2: (no net) -> GND
- C19 pad 1: (no net) -> GND
- C2 pad 2: (no net) -> GND
- C20 pad 2: (no net) -> GND
- C21 pad 2: (no net) -> GND
- C22 pad 2: (no net) -> GND
- C3 pad 2: (no net) -> GND
- C4 pad 2: (no net) -> GND
- C5 pad 2: (no net) -> GND
- C6 pad 2: (no net) -> GND
- C7 pad 2: (no net) -> GND
- C8 pad 1: (no net) -> GND
- C9 pad 2: (no net) -> GND
- D12 pad 1: (no net) -> GND
- D2 pad 2: (no net) -> GND
- D4 pad 2: (no net) -> GND
- D5 pad 1: (no net) -> GND
- D6 pad 1: (no net) -> GND
- D7 pad 1: (no net) -> GND
- D8 pad 1: (no net) -> GND
- D9 pad 1: (no net) -> GND
- I2C pad 1: (no net) -> GND
- ISP pad 6: (no net) -> GND
- J-CV1 pad S: (no net) -> GND
- J-CV1 pad TN: (no net) -> GND
- J-Clk1 pad S: (no net) -> GND
- J-Out1 pad S: (no net) -> GND
- J-Trig1 pad S: (no net) -> GND
- J4 pad 3: (no net) -> GND
- J4 pad 4: (no net) -> GND
- J4 pad 5: (no net) -> GND
- J4 pad 6: (no net) -> GND
- J4 pad 7: (no net) -> GND
- J4 pad 8: (no net) -> GND
- R30 pad 1: (no net) -> GND
- R31 pad 1: (no net) -> GND
- R34 pad 2: (no net) -> GND
- R35 pad 2: (no net) -> GND
- RV1 pad 3: (no net) -> GND
- SERIAL pad 1: (no net) -> GND
- SW1 pad 2: (no net) -> GND
- SW2 pad 2: (no net) -> GND
- SW3 pad 2: (no net) -> GND
- SW4 pad 2: (no net) -> GND
- SW5 pad 2: (no net) -> GND
- SW6 pad 2: (no net) -> GND
- U2 pad 21: (no net) -> GND
- U2 pad 5: (no net) -> GND
- U3 pad 2: (no net) -> GND
Routing:
- net GND: track 0.00 -> 155.5 mm, vias 0 -> 27
- net /MCU328/PD4: track 92.4 -> 77.5 mm
- net +5V: track 280.0 -> 287.4 mm
- net /MCU328/PC2: track 54.8 -> 62.0 mm
- net /MCU328/PC3: track 87.8 -> 93.1 mm
- net /MCU328/PD5: track 46.7 -> 50.2 mm
- net +12V: track 97.6 -> 94.9 mm
- net Net-(R12-Pad2): track 36.3 -> 35.1 mm
- net Net-(J2-Pad5): track 89.6 -> 90.6 mm
- net Net-(C12-Pad2): track 15.3 -> 15.9 mm
- net Net-(C16-Pad2): track 10.4 -> 11.0 mm
- added copper zone on B.Cu, net GND
- added copper zone on F.Cu, net GND
Other:
- board text added: "+12"
- board text added: "-12"
- board text added: "Rev A"
- board text added: "RndSeq"
- board text added: "© Marangisto 2018"
